Commit message: urdf

File: irb2600_description/urdf/irb2600.xacro (robot description, xacro)
@@ -5,4 +5,9 @@
     <!-- links -->
     <link name="${prefix}base_link">
+      <inertial>
+        <origin xyz="0.0 0.0 0.0" rpy="0.0 0.0 0.0"/>
+        <mass value="92.5052"/>
+        <inertia ixx="1.0" ixy="1.0" ixz="1.0" iyy="1.0" iyz="1.0" izz="1.0"/>
+      </inertial>
       <visual>
         <origin xyz="0 0 0" rpy="0 0 0" />
@@ -20,4 +25,9 @@
     </link>
     <link name="${prefix}link_1">
+      <inertial>
+        <origin xyz="0.0 0.0 0.0" rpy="0.0 0.0 0.0"/>
+        <mass value="69.3794"/>
+        <inertia ixx="1.0" ixy="1.0" ixz="1.0" iyy="1.0" iyz="1.0" izz="1.0"/>
+      </inertial>
       <visual>
         <origin xyz="0 0 0" rpy="0 0 0" />
@@ -35,4 +45,9 @@
     </link>
     <link name="${prefix}link_2">
+      <inertial>
+        <origin xyz="0.0 0.0 0.0" rpy="0.0 0.0 0.0"/>
+        <mass value="35.0020"/>
+        <inertia ixx="1.0" ixy="1.0" ixz="1.0" iyy="1.0" iyz="1.0" izz="1.0"/>
+      </inertial>
       <visual>
         <origin xyz="0 0 0" rpy="0 0 0" />
@@ -50,4 +65,9 @@
     </link>
     <link name="${prefix}link_3">
+      <inertial>
+        <origin xyz="0.0 0.0 0.0" rpy="0.0 0.0 0.0"/>
+        <mass value="68.5583"/>
+        <inertia ixx="1.0" ixy="1.0" ixz="1.0" iyy="1.0" iyz="1.0" izz="1.0"/>
+      </inertial>
       <visual>
         <origin xyz="0 0 0" rpy="0 0 0" />
@@ -65,4 +85,9 @@
     </link>
     <link name="${prefix}link_4">
+      <inertial>
+        <origin xyz="0.0 0.0 0.0" rpy="0.0 0.0 0.0"/>
+        <mass value="18.0455"/>
+        <inertia ixx="1.0" ixy="1.0" ixz="1.0" iyy="1.0" iyz="1.0" izz="1.0"/>
+      </inertial>
       <visual>
         <origin xyz="0 0 0" rpy="0 0 0" />
@@ -80,4 +105,9 @@
     </link>
     <link name="${prefix}link_5">
+      <inertial>
+        <origin xyz="0.0 0.0 0.0" rpy="0.0 0.0 0.0"/>
+        <mass value="1.0738"/>
+        <inertia ixx="1.0" ixy="1.0" ixz="1.0" iyy="1.0" iyz="1.0" izz="1.0"/>
+      </inertial>
       <visual>
         <origin xyz="0 0 0" rpy="0 0 0" />
@@ -95,4 +125,9 @@
     </link>
     <link name="${prefix}link_6">
+      <inertial>
+        <origin xyz="0.0 0.0 0.0" rpy="0.0 0.0 0.0"/>
+        <mass value="0.1418"/>
+        <inertia ixx="1.0" ixy="1.0" ixz="1.0" iyy="1.0" iyz="1.0" izz="1.0"/>
+      </inertial>
       <visual>
         <origin xyz="0 0 0" rpy="0 0 0" />
