Commit message: gazebo_update

File: irb2600_description/urdf/gazebo.xacro (robot description, xacro)
@@ -68,25 +68,25 @@
   <!-- Gazebo-specific link properties -->
   <gazebo reference="${prefix}base_link">
-    <material>Gazebo/Orange</material>
+    <material>Gazebo/White</material>
     <turnGravityOff>true</turnGravityOff>
   </gazebo>
   <gazebo reference="${prefix}link_1">
-    <material>Gazebo/Orange</material>
+    <material>Gazebo/White</material>
     <turnGravityOff>true</turnGravityOff>
   </gazebo>
   <gazebo reference="${prefix}link_2">
-    <material>Gazebo/Orange</material>
+    <material>Gazebo/White</material>
     <turnGravityOff>true</turnGravityOff>
   </gazebo>
   <gazebo reference="${prefix}link_3">
-    <material>Gazebo/Orange</material>
+    <material>Gazebo/White</material>
     <turnGravityOff>true</turnGravityOff>
   </gazebo>
   <gazebo reference="${prefix}link_4">
-    <material>Gazebo/Orange</material>
+    <material>Gazebo/White</material>
     <turnGravityOff>true</turnGravityOff>
   </gazebo>
   <gazebo reference="${prefix}link_5">
-    <material>Gazebo/Orange</material>
+    <material>Gazebo/White</material>
     <turnGravityOff>true</turnGravityOff>
   </gazebo>
