Commit message: urdf_xacro_modif

File: irb2600_description/urdf/camera.xacro (robot description, xacro)
@@ -1,76 +1,81 @@
 <?xml version="1.0" ?>
-<robot name="camera" xmlns:xacro="http://ros.org/wiki/xacro">
-	<xacro:property name="PI" value="3.1415926535897931"/>
- <!-- verificar angulo de camera_support -->
-  <link name="camera_support_link">
-    <inertial>
-      <origin
-        xyz="0 0 0"
-        rpy="1.570796327 0 0" />
-      <mass
-        value="0.30915" />
-      <inertia
-        ixx="0.00028972"
-        ixy="-5.7879E-10"
-        ixz="-1.8543E-06"
-        iyy="0.00030737"
-        iyz="1.682E-12"
-        izz="0.00019914" />
-    </inertial>
-    <visual>
-      <origin
-        xyz="0 0 0"
-        rpy="1.570796327 0 0.523598" />
+<robot name="camera" xmlns:xacro="http://wiki.ros.org/xacro">
+  <!-- camera plugin -->
+  <link name="camera">
+    <collision>
+      <origin rpy="0 0 0" xyz="0 0 0"/>
       <geometry>
-        <mesh
-          filename="package://irb120_description/meshes/supports/camera_support.stl" />
-      </geometry>
-      <material name="green"/>
-    </visual>
-    <collision>
-      <origin
-        xyz="0 0 0"
-        rpy="1.570796327 0 0.523598" />
-      <geometry>
-        <mesh
-          filename="package://irb120_description/meshes/supports/camera_support.stl" />
+        <box size="0.1 0.7 0.7"/>
       </geometry>
     </collision>
-  </link>
-  <link name="camera_link">
     <visual>
-      <origin
-        xyz="-0.023 -0.045 -0.0125"
-        rpy="1.570796327 0 1.570796327" />
+      <origin rpy="0 0 0" xyz="0 0 0"/>
       <geometry>
-        <mesh
-          filename="package://irb120_description/meshes/camera.stl" />
+        <box size="0.1 0.7 0.7"/>
       </geometry>
-    <material name="metal_grey"/>
+      <material name="grey"/>
     </visual>
-    <collision>
-      <origin
-        xyz="-0.008 -0.045 -0.0125"
-        rpy="1.570796327 0 1.570796327" />
-      <geometry>
-        <mesh
-          filename="package://irb120_description/meshes/camera.stl" />
-      </geometry>
-    </collision>
     <inertial>
-        <mass value="0.0001" />
-        <origin xyz="0 0 0" rpy="0 0 0"/>
-        <inertia ixx="0.0000001" ixy="0" ixz="0" iyy="0.0000001" iyz="0" izz="0.0000001" />
+      <mass value="0.1"/>
+      <origin rpy="0 0 0" xyz="0 0 0"/>
+      <box_inertia m="0.1" x="0.1" y="0.7" z="0.7"/>
+      <inertia ixx="1e-6" ixy="0" ixz="0" iyy="1e-6" iyz="0" izz="1e-6"/>
     </inertial>
   </link>
-  <joint name="irb120_joint_camera_support" type="fixed">
-    <parent link="tool0"/>
-    <child link="camera_support_link"/>
-    <origin rpy="0 0 0" xyz="0 0 0.008"/>
+  <joint name="camera_optical_joint" type="fixed">
+    <origin rpy="-1.5708 0 -1.5708" xyz="0 0 0"/>
+    <parent link="camera"/>
+    <child link="camera_frame_optical"/>
   </joint>
+  <link name="camera_frame_optical"/>
   <joint name="camera_joint" type="fixed">
-      <origin xyz="0 -0.06 0.095" rpy="0 -1.570796327 1.570796327"/>
-      <parent link="camera_support_link"/>
-      <child link="camera_link"/>
+    <axis xyz="0 0 0"/>
+    <origin rpy="0 1.5708 0" xyz="0.5 0 2.0"/>
+    <parent link="base_link"/>
+    <child link="camera"/>
   </joint>
+  <!-- depth camera -->
+  <gazebo reference="camera">
+    <sensor name="camera1" type="depth">
+      <update_rate>20</update_rate>
+      <camera>
+        <horizontal_fov>1.2</horizontal_fov>
+        <image>
+          <width>640</width>
+          <!--640-->
+          <height>480</height>
+          <!--480-->
+          <format>R8G8B8</format>
+        </image>
+        <clip>
+          <near>0.05</near>
+          <far>30</far>
+        </clip>
+      </camera>
+      <plugin filename="libgazebo_ros_openni_kinect.so" name="camera_controller">
+        <baseline>0.2</baseline>
+        <alwaysOn>false</alwaysOn>
+        <updateRate>0</updateRate>
+        <cameraName>camera1</cameraName>
+        <imageTopicName>/camera1/color/image_raw</imageTopicName>
+        <cameraInfoTopicName>/camera1/color/camera_info</cameraInfoTopicName>
+        <depthImageTopicName>/camera1/depth/image_raw</depthImageTopicName>
+        <depthImageInfoTopicName>/camera1/depth/camera_info</depthImageInfoTopicName>
+        <pointCloudTopicName>/camera1/depth/points</pointCloudTopicName>
+        <frameName>camera_frame_optical</frameName>
+        <pointCloudCutoff>0.5</pointCloudCutoff>
+        <pointCloudCutoffMax>3.0</pointCloudCutoffMax>
+        <distortionK1>0.00000001</distortionK1>
+        <distortionK2>0.00000001</distortionK2>
+        <distortionK3>0.00000001</distortionK3>
+        <distortionT1>0.00000001</distortionT1>
+        <distortionT2>0.00000001</distortionT2>
+        <CxPrime>0</CxPrime>
+        <Cx>0</Cx>
+        <Cy>0</Cy>
+        <focalLength>0</focalLength>
+        <hackBaseline>0</hackBaseline>
+      </plugin>
+    </sensor>
+  </gazebo>
 </robot>

File: irb2600_description/urdf/irb2600_main.xacro (robot description, xacro)
@@ -1,8 +1,13 @@
 <?xml version="1.0" encoding="UTF-8"?>
 <robot name="abb_irb2600_model" xmlns:xacro="http://ros.org/wiki/xacro">
-  <xacro:include filename="$(find irb2600_description)/urdf/irb2600.xacro"/>
+  <xacro:arg name="camera" default="false"/>
+  <xacro:arg name="table" default="false"/>
+  <xacro:arg name="gripper_2f" default="false"/>
+  <xacro:arg name="camera_arm" default="false"/>
+  <xacro:include filename="$(find irb2600_description)/urdf/irb2600_macro.xacro"/>
   <xacro:include filename="$(find irb2600_description)/urdf/gazebo.xacro"/>
   <xacro:abb_irb2600 prefix=""/>
   <link name="world"/>
+  <!-- Fix robot to Gazebo world -->
   <joint name="fixed" type="fixed">
       <parent link="world"/>
@@ -11,3 +16,19 @@
   </joint>
   <xacro:abb_irb2600_gazebo prefix=""/>
+  <!-- table -->
+  <xacro:if value="$(arg table)">
+    <xacro:include filename="$(find irb2600_description)/urdf/table.xacro"/>
+  </xacro:if>
+  <!-- camera -->
+  <xacro:if value="$(arg camera)">
+    <xacro:include filename="$(find irb2600_description)/urdf/camera.xacro"/>
+  </xacro:if>
+  <!-- gripper -->
+  <xacro:if value="$(arg gripper_2f)">
+    <xacro:include filename="$(find irb2600_description)/urdf/gazebo_2f.xacro"/>
+  </xacro:if>
+   <!-- camera arm-->
+  <xacro:if value="$(arg camera_arm)">
+    <xacro:include filename="$(find irb2600_description)/urdf/camera_arm.xacro"/>
+  </xacro:if>
 </robot>

File: irb2600_description/urdf/table.xacro (robot description, xacro)
@@ -7,7 +7,7 @@
 	<link name="table">
 		<visual>
-			<origin rpy="0 0 0" xyz="0.2 0 -0.005"/>
+			<origin rpy="0 0 0" xyz="0.2 0 0.5"/>
 			<geometry>
-			<box size="0.8 1.6 0.01"/>
+			<box size="0.8 1.6 1.01"/>
 			</geometry>
 			<material name="coral"/>
@@ -31,35 +31,8 @@
 		<origin xyz="0 0 0" rpy="0 0 0"/>
 	</joint>
-	<!-- end effect point -->
-	<joint name="end_effect_point" type="fixed">
-		<origin rpy="0 0 -0.6434" xyz="0 0 0.24"/>
-		<parent link="tool0"/>
-		<child link="end_effect_point"/>
+	<joint name="table_base" type="fixed">
+		<parent link="table"/>
+		<child link="base_link"/>
+		<origin xyz="0 0 1.01" rpy="0 0 0"/>
 	</joint>
-	<!-- end effect point -->
-	<link name="end_effect_point">
-		<visual>
-			<origin rpy="0 0 0" xyz="0 0 -0.12"/>
-			<geometry>
-				<box size="0.01 0.01 0.24"/>
-			</geometry>
-			<material name="">
-				<color rgba="0.8 0.0 0.0 1.0"/>
-			</material>
-		</visual>
-		<collision>
-			<origin rpy="0 0 0" xyz="0 0 -0.12"/>
-			<geometry>
-				<box size="0.01 0.01 0.24"/>
-			</geometry>
-			<material name="">
-				<color rgba="0.8 0.0 0.0 1.0"/>
-			</material>
-		</collision>
-		<inertial>
-		<origin rpy="0 0 0" xyz="0.0 0.0 0.0"/>
-		<mass value="0.001"/>
-		<inertia ixx="1.0e-06" ixy="0.0" ixz="0.0" iyy="1.0e-06" iyz="0.0" izz="1.0e-06"/>
-		</inertial>
-	</link>
 </robot>
