Commit message: mass_value

File: irb2600_description/urdf/robot_base.xacro (robot description, xacro)
@@ -24,5 +24,5 @@
 		<inertial>
 			<origin rpy="0 0 0" xyz="0.0 0.0 0.0"/>
-			<mass value="0.001"/>
+			<mass value="120"/>
 			<inertia ixx="1.0e-06" ixy="0.0" ixz="0.0" iyy="1.0e-06" iyz="0.0" izz="1.0e-06"/>
 		</inertial>
