Commit message: update

File: irb2600_description/urdf/camera_l515.xacro (robot description, xacro)
@@ -20,9 +20,9 @@
     <visual>
       <origin
-        xyz="0 0 0"
-        rpy="1.570796327 0 0.523598" />
+        xyz="0.025 -0.06 -0.045"
+        rpy="1.570796327 0 -1.570796327" />
       <geometry>
         <mesh
-          filename="package://irb2600_description/meshes/supports/camera_support.stl" />
+          filename="package://irb2600_description/meshes/supports/cameral515.stl" />
       </geometry>
       <material name="green"/>
@@ -31,12 +31,12 @@
       <origin
         xyz="0 0 0"
-        rpy="1.570796327 0 0.523598" />
+        rpy="1.570796327 0 -1.570796327" />
       <geometry>
         <mesh
-          filename="package://irb2600_description/meshes/supports/camera_support.stl" />
+          filename="package://irb2600_description/meshes/supports/cameral515.stl" />
       </geometry>
     </collision>
   </link>
-  <link name="camera_link">
+  <!--<link name="camera_link">
     <visual>
       <origin
@@ -45,5 +45,5 @@
       <geometry>
         <mesh
-          filename="package://irb2600_description/meshes/camera.stl" />
+          filename="package://irb2600_description/meshes/cameral515_sim.stl"/>
       </geometry>
     <material name="metal_grey"/>
@@ -55,5 +55,5 @@
       <geometry>
         <mesh
-          filename="package://irb2600_description/meshes/camera.stl" />
+          filename="package://irb2600_description/meshes/cameral515_sim.stl" />
       </geometry>
     </collision>
@@ -63,5 +63,5 @@
         <inertia ixx="0.0000001" ixy="0" ixz="0" iyy="0.0000001" iyz="0" izz="0.0000001" />
     </inertial>
-  </link>
+  </link>-->
   <joint name="irb2600_joint_camera_support" type="fixed">
     <parent link="tool0"/>
@@ -69,12 +69,12 @@
     <origin rpy="0 0 -1.570796" xyz="0 0 0.008"/>
   </joint>
-  <joint name="camera_joint" type="fixed">
+  <!--<joint name="camera_joint" type="fixed">
       <origin xyz="0 -0.06 0.095" rpy="0 -1.570796327 1.570796327"/>
       <parent link="camera_support_link"/>
       <child link="camera_link"/>
-  </joint>
+  </joint>-->
   <joint name="camera_optical_joint" type="fixed">
     <origin rpy="-1.5708 0 -1.5708" xyz="0 0 0"/>
-    <parent link="camera_link"/>
+    <parent link="camera_support_link"/>
     <child link="camera_frame_optical"/>
   </joint>
