Commit message: update_gazebo

File: irb2600_description/urdf/irb2600_main.xacro (robot description, xacro)
@@ -2,4 +2,11 @@
 <robot name="abb_irb2600_model" xmlns:xacro="http://ros.org/wiki/xacro">
   <xacro:include filename="$(find irb2600_description)/urdf/irb2600.xacro"/>
+  <xacro:include filename="$(find irb2600_description)/urdf/gazebo.xacro"/>
   <xacro:abb_irb2600 prefix=""/>
+  <link name="world"/>
+  <joint name="fixed" type="fixed">
+      <parent link="world"/>
+      <child link="base_link"/>
+      <origin rpy="0 0 0" xyz="0 0 0"/>
+  </joint>
 </robot>

Commit message: platform_added

File: irb2600_description/urdf/irb2600_main.xacro (robot description, xacro)
@@ -5,18 +5,23 @@
   <xacro:arg name="gripper_2f" default="false"/>
   <xacro:arg name="camera_arm" default="false"/>
+  <xacro:arg name="robot_base" default="false"/>
   <xacro:include filename="$(find irb2600_description)/urdf/irb2600_macro.xacro"/>
   <xacro:include filename="$(find irb2600_description)/urdf/gazebo.xacro"/>
   <xacro:abb_irb2600 prefix=""/>
   <link name="world"/>
-  <!-- Fix robot to Gazebo world -->
+  <!-- Fix robot to Gazebo world
   <joint name="fixed" type="fixed">
       <parent link="world"/>
       <child link="base_link"/>
       <origin rpy="0 0 0" xyz="0 0 0"/>
-  </joint>
+  </joint> -->
   <xacro:abb_irb2600_gazebo prefix=""/>
   <!-- table -->
   <xacro:if value="$(arg table)">
     <xacro:include filename="$(find irb2600_description)/urdf/table.xacro"/>
+  </xacro:if>
+  <!-- robot lab base -->
+  <xacro:if value="$(arg robot_base)">
+    <xacro:include filename="$(find irb2600_description)/urdf/robot_base.xacro"/>
   </xacro:if>
   <!-- camera -->

Commit message: vacuum_gripper_added

File: irb2600_description/urdf/irb2600_main.xacro (robot description, xacro)
@@ -6,14 +6,10 @@
   <xacro:arg name="camera_arm" default="false"/>
   <xacro:arg name="robot_base" default="false"/>
+  <xacro:arg name="vacuum_end" default="false"/>
+  <xacro:arg name="base_vacuum_end" default="false"/>
   <xacro:include filename="$(find irb2600_description)/urdf/irb2600_macro.xacro"/>
   <xacro:include filename="$(find irb2600_description)/urdf/gazebo.xacro"/>
   <xacro:abb_irb2600 prefix=""/>
   <link name="world"/>
-  <!-- Fix robot to Gazebo world
-  <joint name="fixed" type="fixed">
-      <parent link="world"/>
-      <child link="base_link"/>
-      <origin rpy="0 0 0" xyz="0 0 0"/>
-  </joint> -->
   <xacro:abb_irb2600_gazebo prefix=""/>
   <!-- table -->
@@ -25,14 +21,27 @@
     <xacro:include filename="$(find irb2600_description)/urdf/robot_base.xacro"/>
   </xacro:if>
+  <!-- robot vacuum gripper -->
+  <xacro:if value="$(arg vacuum_end)">
+    <xacro:include filename="$(find irb2600_description)/urdf/fixed_world.xacro"/>
+    <xacro:include filename="$(find irb2600_description)/urdf/vacuum_end.xacro"/>
+  </xacro:if>
+  <!-- robot vacuum gripper -->
+  <xacro:if value="$(arg base_vacuum_end)">
+    <xacro:include filename="$(find irb2600_description)/urdf/robot_base.xacro"/>
+    <xacro:include filename="$(find irb2600_description)/urdf/vacuum_end.xacro"/>
+  </xacro:if>
   <!-- camera -->
   <xacro:if value="$(arg camera)">
+    <xacro:include filename="$(find irb2600_description)/urdf/fixed_world.xacro"/>
     <xacro:include filename="$(find irb2600_description)/urdf/camera.xacro"/>
   </xacro:if>
   <!-- gripper -->
   <xacro:if value="$(arg gripper_2f)">
+    <xacro:include filename="$(find irb2600_description)/urdf/fixed_world.xacro"/>
     <xacro:include filename="$(find irb2600_description)/urdf/gazebo_2f.xacro"/>
   </xacro:if>
    <!-- camera arm-->
   <xacro:if value="$(arg camera_arm)">
+    <xacro:include filename="$(find irb2600_description)/urdf/fixed_world.xacro"/>
     <xacro:include filename="$(find irb2600_description)/urdf/camera_arm.xacro"/>
   </xacro:if>

Commit message: wall_updated

File: irb2600_description/urdf/irb2600_main.xacro (robot description, xacro)
@@ -8,4 +8,5 @@
   <xacro:arg name="vacuum_end" default="false"/>
   <xacro:arg name="base_vacuum_end" default="false"/>
+  <xacro:arg name="base_vacuum_end_wall" default="true"/>
   <xacro:include filename="$(find irb2600_description)/urdf/irb2600_macro.xacro"/>
   <xacro:include filename="$(find irb2600_description)/urdf/gazebo.xacro"/>
@@ -26,5 +27,5 @@
     <xacro:include filename="$(find irb2600_description)/urdf/vacuum_end.xacro"/>
   </xacro:if>
-  <!-- robot vacuum gripper -->
+  <!-- robot lab vacuum gripper -->
   <xacro:if value="$(arg base_vacuum_end)">
     <xacro:include filename="$(find irb2600_description)/urdf/robot_base.xacro"/>
@@ -46,3 +47,10 @@
     <xacro:include filename="$(find irb2600_description)/urdf/camera_arm.xacro"/>
   </xacro:if>
+  <!-- robot lab vacuum gripper and wall -->
+  <xacro:if value="$(arg base_vacuum_end_wall)">
+    <xacro:include filename="$(find irb2600_description)/urdf/robot_base.xacro"/>
+    <xacro:include filename="$(find irb2600_description)/urdf/vacuum_end.xacro"/>
+    <xacro:include filename="$(find irb2600_description)/urdf/wall.xacro"/>
+    <xacro:include filename="$(find irb2600_description)/urdf/table.xacro"/>
+  </xacro:if>
 </robot>

File: irb2600_description/urdf/table.xacro (robot description, xacro)
@@ -1,5 +1,5 @@
 <?xml version="1.0" ?>
 <robot name="table" xmlns:xacro="http://ros.org/wiki/xacro">
-	<material name="coral">
+	<material name="coral3">
 		<color rgba="${255/255} ${127/255} ${80/255} 1.0"/>
 	</material>
@@ -7,9 +7,9 @@
 	<link name="table">
 		<visual>
-			<origin rpy="0 0 0" xyz="0.2 0 0.5"/>
+			<origin rpy="0 0 0" xyz="0 2.0 0.405"/>
 			<geometry>
-			<box size="0.8 1.6 1.01"/>
+			<box size="1.5 0.7 0.81"/>
 			</geometry>
-			<material name="coral"/>
+			<material name="coral3"/>
 		</visual>
 		<collision>
@@ -18,5 +18,5 @@
 			<box size="0.8 1.6 0.01"/>
 			</geometry>
-			<material name="coral"/>
+			<material name="coral3"/>
 		</collision>
 		<inertial>
@@ -29,10 +29,5 @@
 		<parent link="world"/>
 		<child link="table"/>
-		<origin xyz="0 0 0" rpy="0 0 0"/>
-	</joint>
-	<joint name="table_base" type="fixed">
-		<parent link="table"/>
-		<child link="base_link"/>
-		<origin xyz="0 0 1.01" rpy="0 0 0"/>
+		<origin xyz="0 0 0" rpy="0 0 -1.57"/>
 	</joint>
 </robot>

Commit message: end_effect_point

File: irb2600_description/urdf/irb2600_main.xacro (robot description, xacro)
@@ -5,5 +5,5 @@
   <xacro:arg name="camera_arm" default="false"/>
   <xacro:arg name="robot_base" default="false"/>
-  <xacro:arg name="vacuum_end" default="false"/>
+  <xacro:arg name="vacuum_end" default="true"/>
   <xacro:arg name="base_vacuum_end" default="false"/>
   <xacro:arg name="base_vacuum_end_wall" default="false"/>

File: irb2600_description/urdf/vacuum_end.xacro (robot description, xacro)
@@ -46,3 +46,26 @@
     <origin rpy="0 0 -1.570796" xyz="0 0 0.0634"/>
   </joint>
+  <!-- end effect point -->
+  <joint name="end_effect_point" type="fixed">
+    <origin rpy="0 0 0" xyz="0 0 0.2472"/>
+    <parent link="tool0"/>
+    <child link="end_effect_point"/>
+  </joint>
+  <!-- end effect point -->
+  <link name="end_effect_point">
+    <visual>
+      <origin rpy="0 0 0" xyz="0 0 -0.1"/>
+      <geometry>
+        <box size="0.002 0.002 0.002"/>
+      </geometry>
+      <material name="">
+        <color rgba="0.8 0.0 0.0 1.0"/>
+      </material>
+    </visual>
+    <!-- <inertial>
+      <origin rpy="0 0 0" xyz="0.0 0.0 0.0"/>
+      <mass value="0.001"/>
+      <inertia ixx="1.0e-06" ixy="0.0" ixz="0.0" iyy="1.0e-06" iyz="0.0" izz="1.0e-06"/>
+    </inertial> -->
+  </link>
 </robot>

Commit message: moveit_vacuum

File: irb2600_description/urdf/irb2600_main.xacro (robot description, xacro)
@@ -5,5 +5,5 @@
   <xacro:arg name="camera_arm" default="false"/>
   <xacro:arg name="robot_base" default="false"/>
-  <xacro:arg name="vacuum_end" default="true"/>
+  <xacro:arg name="vacuum_end" default="false"/>
   <xacro:arg name="base_vacuum_end" default="false"/>
   <xacro:arg name="base_vacuum_end_wall" default="false"/>

File: irb2600_description/urdf/vacuum_end.xacro (robot description, xacro)
@@ -63,9 +63,15 @@
       </material>
     </visual>
-    <!-- <inertial>
+    <!--<collision>
+      <origin rpy="0 0 0" xyz="0 0 -0.1"/>
+      <geometry>
+        <box size="0.002 0.002 0.002"/>
+      </geometry>
+    </collision>-->
+    <inertial>
       <origin rpy="0 0 0" xyz="0.0 0.0 0.0"/>
       <mass value="0.001"/>
       <inertia ixx="1.0e-06" ixy="0.0" ixz="0.0" iyy="1.0e-06" iyz="0.0" izz="1.0e-06"/>
-    </inertial> -->
+    </inertial>
   </link>
 </robot>

Commit message: update

File: irb2600_description/urdf/irb2600_main.xacro (robot description, xacro)
@@ -1,26 +1,23 @@
 <?xml version="1.0" encoding="UTF-8"?>
 <robot name="abb_irb2600_model" xmlns:xacro="http://ros.org/wiki/xacro">
-  <xacro:arg name="camera" default="false"/>
   <xacro:arg name="table" default="false"/>
-  <xacro:arg name="camera_arm" default="false"/>
-  <xacro:arg name="robot_base" default="false"/>
-  <xacro:arg name="vacuum_end" default="true"/>
+  <xacro:arg name="camera_d435" default="false"/>
+  <xacro:arg name="camera_l515" default="false"/>
+  <xacro:arg name="vacuum_end" default="false"/>
   <xacro:arg name="base_vacuum_end" default="false"/>
   <xacro:arg name="base_vacuum_end_wall" default="false"/>
+  <link name="world"/>
+  <!-- Robot base 6 joints -->
   <xacro:include filename="$(find irb2600_description)/urdf/irb2600_macro.xacro"/>
   <xacro:include filename="$(find irb2600_description)/urdf/gazebo.xacro"/>
   <xacro:abb_irb2600 prefix=""/>
-  <link name="world"/>
   <xacro:abb_irb2600_gazebo prefix=""/>
+  <!-- Robot base support -->
   <xacro:include filename="$(find irb2600_description)/urdf/robot_base.xacro"/>
+  <!-- walls around robot -->
   <xacro:include filename="$(find irb2600_description)/urdf/wall.xacro"/>
-  <xacro:include filename="$(find irb2600_description)/urdf/table.xacro"/>
   <!-- table -->
   <xacro:if value="$(arg table)">
     <xacro:include filename="$(find irb2600_description)/urdf/table.xacro"/>
-  </xacro:if>
-  <!-- robot lab base -->
-  <xacro:if value="$(arg robot_base)">
-    <xacro:include filename="$(find irb2600_description)/urdf/robot_base.xacro"/>
   </xacro:if>
   <!-- robot vacuum gripper -->
@@ -28,23 +25,11 @@
     <xacro:include filename="$(find irb2600_description)/urdf/vacuum_end.xacro"/>
   </xacro:if>
-  <!-- robot lab vacuum gripper -->
-  <xacro:if value="$(arg base_vacuum_end)">
-    <xacro:include filename="$(find irb2600_description)/urdf/robot_base.xacro"/>
-    <xacro:include filename="$(find irb2600_description)/urdf/vacuum_end.xacro"/>
+  <!-- camera_d435 -->
+  <xacro:if value="$(arg camera_d435)">
+    <xacro:include filename="$(find irb2600_description)/urdf/camera_d435.xacro"/>
   </xacro:if>
-  <!-- camera -->
-  <xacro:if value="$(arg camera)">
-    <xacro:include filename="$(find irb2600_description)/urdf/camera.xacro"/>
-  </xacro:if>
-   <!-- camera arm-->
-  <xacro:if value="$(arg camera_arm)">
-    <xacro:include filename="$(find irb2600_description)/urdf/camera_arm.xacro"/>
-  </xacro:if>
-  <!-- robot lab vacuum gripper and wall -->
-  <xacro:if value="$(arg base_vacuum_end_wall)">
-    <xacro:include filename="$(find irb2600_description)/urdf/robot_base.xacro"/>
-    <xacro:include filename="$(find irb2600_description)/urdf/vacuum_end.xacro"/>
-    <xacro:include filename="$(find irb2600_description)/urdf/wall.xacro"/>
-    <xacro:include filename="$(find irb2600_description)/urdf/table.xacro"/>
+   <!-- camera_l515-->
+  <xacro:if value="$(arg camera_l515)">
+    <xacro:include filename="$(find irb2600_description)/urdf/camera_l515.xacro"/>
   </xacro:if>
 </robot>

Commit message: Se realizo el urdf del nuevo end effector y se realizo el movveit, ademas se cambio ciertos parametros de la mesa y el color de las paredes para que se vea mas amigable

File: irb2600_description/urdf/irb2600_main.xacro (robot description, xacro)
@@ -5,4 +5,5 @@
   <xacro:arg name="camera_l515" default="false"/>
   <xacro:arg name="vacuum_end" default="false"/>
+  <xacro:arg name="ee_marker" default="true"/>
   <xacro:arg name="base_vacuum_end" default="false"/>
   <xacro:arg name="base_vacuum_end_wall" default="false"/>
@@ -33,3 +34,7 @@
     <xacro:include filename="$(find irb2600_description)/urdf/camera_l515.xacro"/>
   </xacro:if>
+  <!-- robot marcador end effector -->
+  <xacro:if value="$(arg ee_marker)">
+    <xacro:include filename="$(find irb2600_description)/urdf/ee_marker.xacro"/>
+  </xacro:if>
 </robot>

File: irb2600_description/urdf/table.xacro (robot description, xacro)
@@ -2,12 +2,12 @@
 <robot name="table" xmlns:xacro="http://ros.org/wiki/xacro">
 	<material name="coral3">
-		<color rgba="${255/255} ${127/255} ${80/255} 1.0"/>
+		<color rgba="${255/255} ${255/255} ${255/255} 1.0"/>
 	</material>
 	<!-- HERE you can change the position of the robot in the table -->
 	<link name="table">
 		<visual>
-			<origin rpy="0 0 0" xyz="0 2.0 0.405"/>
+			<origin rpy="0 0 0" xyz="0 1.20 0"/>
 			<geometry>
-			<box size="1.5 0.7 0.81"/>
+			<box size="1.3 0.7 0.82"/>
 			</geometry>
 			<material name="coral3"/>
@@ -29,5 +29,5 @@
 		<parent link="world"/>
 		<child link="table"/>
-		<origin xyz="0 0 0" rpy="0 0 -1.57"/>
+		<origin xyz="0 0 0.41" rpy="0 0 -1.57"/>
 	</joint>
 	<gazebo reference="table">

File: irb2600_description/urdf/wall.xacro (robot description, xacro)
@@ -2,5 +2,5 @@
 <robot name="wall" xmlns:xacro="http://ros.org/wiki/xacro">
 	<material name="coral4">
-		<color rgba="${255/255} ${127/255} ${80/255} 1.0"/>
+		<color rgba="${0/255} ${0/255} ${0/255} 0.5"/>
 	</material>
 	<material name="transparent">

File: moveit_configuration/irb2600_write_moveit/config/gazebo_abb_irb2600_model.urdf (robot description, URDF)
Before this commit: robot abb_irb2600_model, 16 links, 15 joints
Links:
- added link ee, mass 0.0453532792285496; collision mesh filename=package://irb2600_description/meshes/supports/ee_marker.STL; visual mesh filename=package://irb2600_description/meshes/supports/ee_marker.STL
- added link end_effect_point, mass 0.1; collision box size=0.002 0.002 0.002; visual box size=0.01 0.01 0.01
- link table: geometry collision box size=1.5 0.7 0.81; visual box size=1.3 0.7 0.82
Joints:
- added joint end_effect_point: type fixed, parent tool0, child end_effect_point, origin xyz=0 0 0 rpy=0 0 0
- added joint irb2600_ee_joint: type fixed, parent tool0, child ee, origin xyz=0 0 0 rpy=1.57 0 0
- joint table_j: origin xyz=0 0 0 rpy=0 0 -1.57 -> xyz=0 0 0.41 rpy=0 0 -1.57
