Commit message: gazeboedited_urdf

File: irb2600_description/urdf/table.xacro (robot description, xacro)
@@ -14,7 +14,7 @@
 		</visual>
 		<collision>
-			<origin rpy="0 0 0" xyz="0.2 0 -0.005"/>
+			<origin rpy="0 0 0" xyz="0 2.0 0.405"/>
 			<geometry>
-			<box size="0.8 1.6 0.01"/>
+			<box size="1.5 0.7 0.81"/>
 			</geometry>
 			<material name="coral3"/>
@@ -26,8 +26,11 @@
 		</inertial>
   	</link>
-	<joint name="table" type="fixed">
+	<joint name="table_j" type="fixed">
 		<parent link="world"/>
 		<child link="table"/>
 		<origin xyz="0 0 0" rpy="0 0 -1.57"/>
 	</joint>
+	<gazebo reference="table">
+    <material>Gazebo/Wood</material>
+  	</gazebo>
 </robot>

File: irb2600_description/urdf/wall.xacro (robot description, xacro)
@@ -86,3 +86,6 @@
 		<origin xyz="0 0 0" rpy="0 0 -1.57"/>
 	</joint>
+	<gazebo reference="wall_left">
+    <material>Gazebo/GreyTransparent</material>
+  	</gazebo>
 </robot>

Commit message: Se probo la escritura del abb, y el marker para su visualizacion en rviz

File: irb2600_description/urdf/table.xacro (robot description, xacro)
@@ -14,7 +14,7 @@
 		</visual>
 		<collision>
-			<origin rpy="0 0 0" xyz="0 2.0 0.405"/>
+			<origin rpy="0 0 0" xyz="0 1.20 0"/>
 			<geometry>
-			<box size="1.5 0.7 0.81"/>
+			<box size="1.3 0.7 0.82"/>
 			</geometry>
 			<material name="coral3"/>

File: moveit_configuration/irb2600_write_moveit/config/gazebo_abb_irb2600_model.urdf (robot description, URDF)
Before this commit: robot abb_irb2600_model, 18 links, 17 joints
Links:
- link table: geometry collision box size=1.3 0.7 0.82; visual box size=1.3 0.7 0.82
